File: olliw-stm32-based/rx-board-01/mLRS-rx-board01-v014.brd (EAGLE design)
At the start: 40.6 x 21.6 mm, 41 parts, among them IC1 stm32F103CX, IC2 NCP1117ST33, IC3 SX1280, IC4 SX1280, Q1 CSTCE8M00G55-R0, Q2 CRYSTAL52MHZ, Q3 CRYSTAL52MHZ, SW1 SWITCH-SMD-TOP-2P6X1P6

Commit message: ups
Parts:
- added IC5: 74AHC1G86, # stdlib:SOT23-5-VER1
- added R3: 10k, rcl:R0402
Connections:
- new net OUT: IC5.4, JP3.1
- new net XOR: IC1.38, IC5.1, R3.2
- net 3.3V: now also IC5.5
- net GND: now also IC5.3, R3.1
- net UART1_TX: now also IC5.2; no longer JP3.1
Routing:
- net XOR: track 0.00 -> 13.1 mm, vias 0 -> 1
- net 3.3V: track 94.1 -> 102.7 mm
- net OUT: track 0.00 -> 2.19 mm
- net UART1_TX: track 14.7 -> 16.3 mm, vias 0 -> 1
- net GND: vias 80 -> 81
Other:
- board text added: "v0.14 rev00"
- board text removed: "v0.13 rev00"

Commit message: tidy
Parts:
- added TP3: TPTP08R, testpad:TP08R
- IC1: value stm32F103CX -> STM32F103CB
- IM1, IM2: value SX-IMPEDANCE-MATCH -> 2450FM07D0034
- Q2, Q3: value CRYSTAL52MHZ -> FW520WFMT1
- moved C5 0.32 mm to (35.4, 9.37)
- moved C6 0.32 mm to (35.4, 11.6)
- moved C14 0.16 mm to (16.0, 23.8)
- moved LED1 0.16 mm to (41.3, 5.40)
- moved LED2 0.16 mm to (41.3, 6.99)
- moved R1 0.16 mm to (37.9, 5.40)
- moved R2 0.16 mm to (37.9, 6.99)
- moved C19 0.16 mm to (16.0, 13.7)
- renumbered C13 to C12, JP1 to PH-SWD, JP2 to PH-SERIAL, JP3 to PH-OUT, SW1 to S1, U$11 to UFL2, U$9 to UFL1
Connections:
- net N$16 renamed UFL1
- removed net USBDM: IC1.32
- new net N$9: IC1.32, TP3.TP
- net GND: now also IC1.3, IC1.4
Routing:
- net N$9: track 0.00 -> 5.95 mm
- net VCC: track 24.6 -> 25.3 mm
- net 3.3V: track 102.7 -> 103.3 mm
- net GND: vias 81 -> 82
Other:
- board text added: "mLRS"
