File: olliw-stm32-based/rx-board-01/mLRS-rx-board01-v014.sch (EAGLE design)
At the start: 41 parts, among them IC1 stm32F103CX, IC2 NCP1117ST33, IC3 SX1280, IC4 SX1280, Q1 CSTCE8M00G55-R0, Q2 CRYSTAL52MHZ, Q3 CRYSTAL52MHZ, SW1 SWITCH-SMD-TOP-2P6X1P6

Commit message: ups
Parts:
- added IC5: 74AHC1G86, # stdlib:74AHC1G86
- added R3: 10k, rcl:R-EU_R0402
Connections:
- new net OUT: IC5.O, JP3.1
- new net XOR: IC1PORTA_H.PA15, IC5.I0, R3.2
- net 3.3V: now also IC5.VCC
- net GND: now also IC5.GND, R3.1
- net UART1_TX: now also IC5.I1; no longer JP3.1
Changed lines of the file:
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@@
 <part name="GND30" library="# supply1" deviceset="GND" device=""/>
 <part name="R2" library="rcl" deviceset="R-EU_" device="R0402" value="2.2k"/>
-<part name="GND12" library="# supply1" deviceset="GND" device=""/>
 <part name="GND31" library="# supply1" deviceset="GND" device=""/>
 <part name="JP2" library="# stdlib" deviceset="PINHEAD_3X2" device="WITHOUT"/>
@@
 <part name="P+7" library="# SparkFun2" deviceset="3.3V" device=""/>
 <part name="GND4" library="# supply1" deviceset="GND" device=""/>
+<part name="GND37" library="# supply1" deviceset="GND" device=""/>
+<part name="P+8" library="# SparkFun2" deviceset="3.3V" device=""/>
+<part name="IC5" library="# stdlib" deviceset="74AHC1G86" device=""/>
+<part name="R3" library="rcl" deviceset="R-EU_" device="R0402" value="10k"/>
+<part name="GND12" library="# supply1" deviceset="GND" device=""/>
 </parts>
 <sheets>
@@
 The project web page is http://www.olliw.eu/.</text>
 <text x="96.52" y="86.36" size="1.778" layer="91">boot1</text>
+<text x="106.68" y="30.48" size="1.778" layer="91">dummy</text>
 <text x="96.52" y="78.74" size="1.778" layer="91">dummy</text>
-<text x="106.68" y="30.48" size="1.778" layer="91">dummy</text>
 </plain>
 <instances>
@@
 <instance part="GND30" gate="1" x="205.74" y="45.72"/>
 <instance part="R2" gate="G$1" x="187.96" y="50.8"/>
-<instance part="GND12" gate="1" x="121.92" y="78.74" rot="R90"/>
 <instance part="GND31" gate="1" x="121.92" y="30.48" rot="R90"/>
 <instance part="JP2" gate="G$1" x="187.96" y="-2.54" rot="MR180"/>
@@
 <instance part="P+7" gate="G$1" x="251.46" y="68.58"/>
 <instance part="GND4" gate="1" x="251.46" y="48.26"/>
+<instance part="GND37" gate="1" x="160.02" y="88.9"/>
+<instance part="P+8" gate="G$1" x="160.02" y="114.3"/>
+<instance part="IC5" gate="G$1" x="160.02" y="104.14" rot="MR0"/>
+<instance part="R3" gate="G$1" x="167.64" y="93.98"/>
+<instance part="GND12" gate="1" x="121.92" y="78.74" rot="R90"/>
 </instances>
 <busses>
@@
 </segment>
 <segment>
-<pinref part="IC1" gate="PORTB_L" pin="PB5"/>
-<wire x1="93.98" y1="78.74" x2="119.38" y2="78.74" width="0.1524" layer="91"/>
-<pinref part="GND12" gate="1" pin="GND"/>
-</segment>
-<segment>
 <pinref part="IC1" gate="PORTA_H" pin="PA12"/>
 <label x="96.52" y="30.48" size="1.778" layer="95"/>
@@
 <wire x1="251.46" y1="50.8" x2="251.46" y2="53.34" width="0.1524" layer="91"/>
 <junction x="251.46" y="53.34"/>
+</segment>
+<segment>
+<pinref part="GND37" gate="1" pin="GND"/>
+<pinref part="IC5" gate="G$1" pin="GND"/>
+<wire x1="160.02" y1="91.44" x2="160.02" y2="93.98" width="0.1524" layer="91"/>
+<pinref part="R3" gate="G$1" pin="1"/>
+<wire x1="160.02" y1="93.98" x2="160.02" y2="96.52" width="0.1524" layer="91"/>
+<wire x1="162.56" y1="93.98" x2="160.02" y2="93.98" width="0.1524" layer="91"/>
+<junction x="160.02" y="93.98"/>
+</segment>
+<segment>
+<pinref part="IC1" gate="PORTB_L" pin="PB5"/>
+<pinref part="GND12" gate="1" pin="GND"/>
+<wire x1="93.98" y1="78.74" x2="119.38" y2="78.74" width="0.1524" layer="91"/>
 </segment>
 </net>
@@
 <junction x="251.46" y="66.04"/>
 </segment>
+<segment>
+<pinref part="P+8" gate="G$1" pin="3.3V"/>
+<pinref part="IC5" gate="G$1" pin="VCC"/>
+<wire x1="160.02" y1="114.3" x2="160.02" y2="111.76" width="0.1524" layer="91"/>
+</segment>
 </net>
 <net name="N$5" class="0">
@@
 </segment>
 <segment>
-<pinref part="JP3" gate="G$1" pin="1"/>
-<wire x1="246.38" y1="0" x2="223.52" y2="0" width="0.1524" layer="91"/>
-<label x="223.52" y="0" size="1.778" layer="95"/>
+<wire x1="190.5" y1="101.6" x2="165.1" y2="101.6" width="0.1524" layer="91"/>
+<pinref part="IC5" gate="G$1" pin="I1"/>
+<wire x1="170.18" y1="101.6" x2="165.1" y2="101.6" width="0.1524" layer="91"/>
+<label x="182.88" y="101.6" size="1.778" layer="95"/>
 </segment>
 </net>
@@
 </segment>
 </net>
+<net name="OUT" class="0">
+<segment>
+<pinref part="IC5" gate="G$1" pin="O"/>
+<wire x1="154.94" y1="104.14" x2="142.24" y2="104.14" width="0.1524" layer="91"/>
+<label x="142.24" y="104.14" size="1.778" layer="95"/>
+</segment>
+<segment>
+<pinref part="JP3" gate="G$1" pin="1"/>
+<wire x1="246.38" y1="0" x2="223.52" y2="0" width="0.1524" layer="91"/>
+<label x="223.52" y="0" size="1.778" layer="95"/>
+</segment>
+</net>
+<net name="XOR" class="0">
+<segment>
+<wire x1="175.26" y1="106.68" x2="190.5" y2="106.68" width="0.1524" layer="91"/>
+<wire x1="175.26" y1="106.68" x2="175.26" y2="93.98" width="0.1524" layer="91"/>
+<wire x1="175.26" y1="93.98" x2="172.72" y2="93.98" width="0.1524" layer="91"/>
+<wire x1="165.1" y1="106.68" x2="175.26" y2="106.68" width="0.1524" layer="91"/>
+<junction x="175.26" y="106.68"/>
+<pinref part="IC5" gate="G$1" pin="I0"/>
+<label x="182.88" y="106.68" size="1.778" layer="95"/>
+<pinref part="R3" gate="G$1" pin="2"/>
+</segment>
+<segment>
+<wire x1="93.98" y1="22.86" x2="109.22" y2="22.86" width="0.1524" layer="91"/>
+<label x="101.6" y="22.86" size="1.778" layer="95"/>
+<pinref part="IC1" gate="PORTA_H" pin="PA15"/>
+</segment>
+</net>

Commit message: tidy
Parts:
- removed SW1: SWITCH-SMD-TOP-2P6X1P6, # stdlib:SWITCH-SMD-TOP-2P6X1P6
- removed U$11, U$9: IPEX-UFL, # stdlib:IPEX-UFL
- added S1: SWITCH-SMD-TOP-2P6X1P6, # stdlib:SWITCH-SMD-TOP-2P6X1P6
- added TP3: TPTP08R, testpad:TPTP08R
- added UFL1, UFL2: IPEX-UFL, # stdlib:IPEX-UFL
- IC1: value stm32F103CX -> STM32F103CB
- IM1, IM2: value SX-IMPEDANCE-MATCH -> 2450FM07D0034
- Q2, Q3: value CRYSTAL52MHZ -> FW520WFMT1
- renumbered C13 to C12, JP1 to PH-SWD, JP2 to PH-SERIAL, JP3 to PH-OUT
Connections:
- removed net N$16: IM1.OUT, U$9.1
- removed net USBDM: IC1PORTA_H.PA11
- new net N$9: IC1PORTA_H.PA11, TP3.TP
- new net UFL1: IM1.OUT, UFL1.1
- net BUTTON: now also S1.3, S1.4; no longer SW1.3, SW1.4
- net GND: now also IC1PORTC.PC14, IC1PORTC.PC15, S1.1, S1.2, UFL1.2, UFL1.3, UFL2.2, UFL2.3; no longer SW1.1, SW1.2, U$11.2, U$11.3, U$9.2, U$9.3
- net N$18: now also UFL2.1; no longer U$11.1
Other:
- note added: "22. Dez. 2021"
- note added: "Schaltplan v0.14"
- note added: "mLRS Rx Board01"
- note removed: "14. Apr. 2021"
- note removed: "OpenTx S.Port Bridge"
- note removed: "Schaltplan v0.40"
- moved on the sheet: C14, C15, C16, C17, C18, C19, C20, C21, C22, C23, IC3, IC4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
