File: olliw-stm32-based/rx-board-01/mLRS-rx-board01-v014-01.brd (EAGLE design)
At the start: 40.6 x 21.6 mm, 44 parts, among them IC1 STM32F103CB, IC2 NCP1117ST33, IC3 SX1280, IC4 SX1280, IC5 74AHC1G86, Q1 CSTCE8M00G55-R0, Q2 FW520WFMT1, Q3 FW520WFMT1

Commit message: rx board01 v014 rev01
Parts:
- moved IM2 0.24 mm to (10.6, 9.60)
- moved IM1 0.08 mm to (10.6, 19.8)
Other:
- board text added: "v0.14 rev01"
- board text removed: "v0.14 rev00"
Changed lines of the file:
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@@
 <layers>
 <layer number="1" name="Top" color="4" fill="1" visible="yes" active="yes"/>
-<layer number="16" name="Bottom" color="1" fill="1" visible="no" active="yes"/>
+<layer number="16" name="Bottom" color="1" fill="1" visible="yes" active="yes"/>
 <layer number="17" name="Pads" color="2" fill="1" visible="yes" active="yes"/>
 <layer number="18" name="Vias" color="2" fill="1" visible="yes" active="yes"/>
@@
 <layer number="20" name="Dimension" color="15" fill="1" visible="yes" active="yes"/>
 <layer number="21" name="tPlace" color="7" fill="1" visible="yes" active="yes"/>
-<layer number="22" name="bPlace" color="7" fill="1" visible="no" active="yes"/>
+<layer number="22" name="bPlace" color="7" fill="1" visible="yes" active="yes"/>
 <layer number="23" name="tOrigins" color="15" fill="1" visible="yes" active="yes"/>
-<layer number="24" name="bOrigins" color="15" fill="1" visible="no" active="yes"/>
-<layer number="25" name="tNames" color="7" fill="1" visible="no" active="yes"/>
-<layer number="26" name="bNames" color="7" fill="1" visible="no" active="yes"/>
-<layer number="27" name="tValues" color="7" fill="1" visible="yes" active="yes"/>
+<layer number="24" name="bOrigins" color="15" fill="1" visible="yes" active="yes"/>
+<layer number="25" name="tNames" color="7" fill="1" visible="yes" active="yes"/>
+<layer number="26" name="bNames" color="7" fill="1" visible="yes" active="yes"/>
+<layer number="27" name="tValues" color="7" fill="1" visible="no" active="yes"/>
 <layer number="28" name="bValues" color="7" fill="1" visible="no" active="yes"/>
 <layer number="29" name="tStop" color="7" fill="3" visible="yes" active="yes"/>
-<layer number="30" name="bStop" color="7" fill="6" visible="no" active="yes"/>
+<layer number="30" name="bStop" color="7" fill="6" visible="yes" active="yes"/>
 <layer number="31" name="tCream" color="7" fill="4" visible="no" active="yes"/>
 <layer number="32" name="bCream" color="7" fill="5" visible="no" active="yes"/>
 <layer number="33" name="tFinish" color="6" fill="3" visible="yes" active="yes"/>
-<layer number="34" name="bFinish" color="6" fill="6" visible="no" active="yes"/>
+<layer number="34" name="bFinish" color="6" fill="6" visible="yes" active="yes"/>
 <layer number="35" name="tGlue" color="7" fill="4" visible="no" active="yes"/>
 <layer number="36" name="bGlue" color="7" fill="5" visible="no" active="yes"/>
@@
 <layer number="38" name="bTest" color="7" fill="1" visible="no" active="yes"/>
 <layer number="39" name="tKeepout" color="4" fill="11" visible="yes" active="yes"/>
-<layer number="40" name="bKeepout" color="1" fill="11" visible="no" active="yes"/>
+<layer number="40" name="bKeepout" color="1" fill="11" visible="yes" active="yes"/>
 <layer number="41" name="tRestrict" color="4" fill="10" visible="yes" active="yes"/>
-<layer number="42" name="bRestrict" color="1" fill="10" visible="no" active="yes"/>
+<layer number="42" name="bRestrict" color="1" fill="10" visible="yes" active="yes"/>
 <layer number="43" name="vRestrict" color="2" fill="10" visible="yes" active="yes"/>
 <layer number="44" name="Drills" color="7" fill="1" visible="no" active="yes"/>
@@
 <layer number="50" name="dxf" color="7" fill="1" visible="no" active="no"/>
 <layer number="51" name="tDocu" color="7" fill="1" visible="yes" active="yes"/>
-<layer number="52" name="bDocu" color="7" fill="1" visible="no" active="yes"/>
+<layer number="52" name="bDocu" color="7" fill="1" visible="yes" active="yes"/>
 <layer number="53" name="tGND_GNDA" color="7" fill="9" visible="no" active="no"/>
 <layer number="54" name="bGND_GNDA" color="1" fill="9" visible="no" active="no"/>
@@
 <layer number="120" name="Descript" color="7" fill="1" visible="no" active="yes"/>
 <layer number="121" name="_tsilk" color="7" fill="1" visible="yes" active="yes"/>
-<layer number="122" name="_bsilk" color="7" fill="1" visible="no" active="yes"/>
+<layer number="122" name="_bsilk" color="7" fill="1" visible="yes" active="yes"/>
 <layer number="123" name="tTestmark" color="7" fill="1" visible="no" active="yes"/>
 <layer number="124" name="bTestmark" color="7" fill="1" visible="no" active="yes"/>
@@
 <text x="7.62" y="23.01875" size="1.6764" layer="25" font="vector" ratio="15" rot="SR0" align="bottom-center">mLRS</text>
 <text x="30.1625" y="9.8425" size="0.8128" layer="25" font="vector" ratio="15" rot="SR0" align="top-center">v0.14
-rev00</text>
+rev01</text>
+<circle x="32.385" y="20.16125" radius="0.254" width="0.254" layer="21"/>
+<circle x="12.144375" y="7.699375" radius="0.254" width="0.254" layer="21"/>
+<circle x="12.144375" y="17.859375" radius="0.254" width="0.254" layer="21"/>
+<circle x="5.23875" y="21.351875" radius="0.254" width="0.254" layer="21"/>
+<circle x="5.23875" y="11.191875" radius="0.254" width="0.254" layer="21"/>
 </plain>
 <attributes>
@@
 <attribute name="VALUE" x="23.1775" y="5.11175" size="0.0254" layer="27"/>
 </element>
-<element name="IM1" library="# stdlib" package="SX-IMPEDANCE-MATCH" value="2450FM07D0034" x="10.63625" y="19.764375" smashed="yes" rot="R180">
-<attribute name="NAME" x="10.85375" y="18.770625" size="0.8128" layer="25" font="vector" rot="R180"/>
-</element>
-<element name="IM2" library="# stdlib" package="SX-IMPEDANCE-MATCH" value="2450FM07D0034" x="10.795" y="9.604375" smashed="yes" rot="R180">
-<attribute name="NAME" x="11.0125" y="8.610625" size="0.8128" layer="25" font="vector" rot="R180"/>
+<element name="IM1" library="# stdlib" package="SX-IMPEDANCE-MATCH" value="2450FM07D0034" x="10.556875" y="19.764375" smashed="yes" rot="R180">
+<attribute name="NAME" x="10.774375" y="18.770625" size="0.8128" layer="25" font="vector" rot="R180"/>
+</element>
+<element name="IM2" library="# stdlib" package="SX-IMPEDANCE-MATCH" value="2450FM07D0034" x="10.556875" y="9.604375" smashed="yes" rot="R180">
+<attribute name="NAME" x="10.774375" y="8.610625" size="0.8128" layer="25" font="vector" rot="R180"/>
 </element>
 <element name="S1" library="# stdlib" package="TACTILE-SWITCH-SMD-TOP-2P6X1X6" value="SWITCH-SMD-TOP-2P6X1P6" x="35.71875" y="23.65375" smashed="yes" rot="R180"/>
@@
 <contactref element="IM2" pad="1"/>
 <wire x1="12.2875" y1="9.5925" x2="11.4625" y2="9.5925" width="0.254" layer="1"/>
-<wire x1="11.4625" y1="9.5925" x2="11.395" y2="9.604375" width="0.1524" layer="1"/>
+<wire x1="11.4625" y1="9.5925" x2="11.156875" y2="9.604375" width="0.1524" layer="1"/>
 </signal>
 <signal name="N$7">
@@
 <contactref element="IM1" pad="1"/>
 <wire x1="12.2875" y1="19.7525" x2="11.30375" y2="19.7525" width="0.254" layer="1"/>
-<wire x1="11.30375" y1="19.7525" x2="11.23625" y2="19.764375" width="0.1524" layer="1"/>
+<wire x1="11.30375" y1="19.7525" x2="11.156875" y2="19.764375" width="0.1524" layer="1"/>
 </signal>
 <signal name="UART2_RX">
@@
 <contactref element="IM1" pad="2"/>
 <contactref element="UFL1" pad="1"/>
-<wire x1="10.03625" y1="19.764375" x2="8.535" y2="19.764375" width="0.254" layer="1"/>
+<wire x1="9.956875" y1="19.764375" x2="8.535" y2="19.764375" width="0.254" layer="1"/>
 </signal>
 <signal name="N$18">
 <contactref element="IM2" pad="2"/>
 <contactref element="UFL2" pad="1"/>
-<wire x1="10.195" y1="9.604375" x2="8.535" y2="9.604375" width="0.254" layer="1"/>
+<wire x1="9.956875" y1="9.604375" x2="8.535" y2="9.604375" width="0.254" layer="1"/>
 </signal>
 <signal name="N$17">
