File: olliw-stm32-based/tx-module-02/mLRS-tx-dualE28-top-v042.brd (EAGLE design)
At the start: 40 x 58.7 mm, 42 parts, among them IC1 STM32G491RC-TQPF64, IC2 E28-2G4M27S, IC3 E28-2G4M27S, IC4 ESP-TTG0-MICROESP32-TTGO-MICRO, IC5 BT HC06, Q1 CSTCE8M00G55-R0, SW1 JOYSTICK-5WAY

Commit message: tx-module02, E28dual board updated to v042 design
Parts:
- removed C17: 10u, rcl:C0603
- removed R8: 2.2k, rcl:R0402
- added C6, C8: 100n, rcl:C0402
- added C7: 10u, rcl:C0603
- added D2: BAT54J, diode:SOD110-R
- added PH-CON2B: PINHEAD_2X1, # stdlib:PINHEAD_2X1
- added R10, R13: 4.7k, rcl:R0402
- added R11, R6: 2.2k, rcl:R0402
- added R12: 1k, rcl:R0402
- added R14, R15: 10k, rcl:R0402
- added T1: FET-NSOT23, # stdlib:SOT23
- added TP1, TP2, TP3: TPB1,27, testpad:B1,27
- C1: device rcl:C0603 -> rcl:C0402
- C13: value 100n -> 10u; device rcl:C0402 -> rcl:C0603
- C15: value 10u -> 100n; device rcl:C0603 -> rcl:C0402
- C16: device rcl:C0402 -> rcl:C0603
- C2: value 100n -> 47u; device rcl:C0603 -> rcl:C1210
- C3: value 100n -> 47u; device rcl:C0402 -> rcl:C1206K
- C4: value 47u -> 100n; device rcl:C1210 -> rcl:C0402
- C5: value 47u -> 10u; device rcl:C1206K -> rcl:C0603
- IC4: value ESP-TTG0-MICROESP32-TTGO-MICRO -> VREG-5PIN-EN1SOT-89-5; device # stdlib:ESP32-TTGO-MICRO -> # stdlib:SOT-89-5
- IC5: value BT HC06 -> ESP-TTG0-MICROESP32-TTGO-MICRO; device # SerialPortBluetooth:BT_HC05_BASIC -> # stdlib:ESP32-TTGO-MICRO
- moved C1 42.1 mm to (25.5, 12.5), flipped to the bottom, turned to 180 degrees
- moved C2 37.1 mm to (25.9, 15.4), turned to 180 degrees
- moved C15 29.8 mm to (34.6, 54.5), turned to 180 degrees
- moved C3 23.7 mm to (13.8, 33.2), flipped to the top
- moved C4 21.4 mm to (11.3, 30.6), turned to 90 degrees
- moved C13 17.1 mm to (11.0, 47.8), flipped to the top, turned to 180 degrees
- moved C16 15.9 mm to (17.9, 51.6), turned to 90 degrees
- moved IC4 15.9 mm to (14.1, 51.6), turned to 180 degrees
- moved C14 12.1 mm to (14.1, 47.8), turned to 0 degrees
- moved IC5 7.03 mm to (29.4, 45.4)
- moved C5 4.01 mm to (11.1, 36.4), turned to 270 degrees
- moved R7 1.59 mm to (19.4, 23.0)
- moved Q1 0.48 mm to (11.3, 27.1)
- moved C10 0.32 mm to (27.3, 34.8)
- moved R1 0.16 mm to (7.94, 19.4)
- renumbered PH-BOTCON1 to PH-CON1, PH-BOTCON2 to PH-CON2
Connections:
- removed net POS_1: IC1.3, SW1.4
- removed net POS_2: IC1.2, SW1.1
- removed net POS_3: IC1.4, SW1.2
- removed net POS_4: IC1.11, SW1.3
- removed net POS_5: IC1.10, SW1.6
- new net 2.8V: C15.1, C16.1, IC4.5, IC5.2
- new net 5V: C13.1, C14.1, IC4.1, IC4.3, IC4.4, PH-CON1.1
- new net BUZ-: D2.A, T1.3, TP3.TP
- new net DTR: IC1.3, PH-CON2B.2
- new net FAN: IC1.58, R14.1, TP1.TP
- new net N$2: R14.2, R15.2, T1.1
- new net POS_CENTER: IC1.2, SW1.2
- new net POS_DOWN: IC1.10, R12.2, R13.1, SW1.6
- new net POS_LEFT: R11.2, R12.1, SW1.3
- new net POS_RIGHT: R10.2, R11.1, SW1.4
- new net POS_UP: R10.1, SW1.1
- new net RTS: IC1.11, PH-CON2B.1
- net 3.3V: now also C6.1, C7.1, C8.1, D2.C, IC1.28, R13.2, R6.2; no longer C14.1, C15.1, C16.1, C17.1, C4.1, IC4.2, IC5.12, R8.2
- net ESP_GPIO0: now also IC1.25, IC5.25; no longer IC1.24, IC4.25
- net ESP_LED: now also IC5.16; no longer IC4.16
- net ESP_RESET: now also IC5.3; no longer IC4.3
- net ESP_UART3_RX: now also IC5.35; no longer IC4.34, IC5.1
- net ESP_UART3_TX: now also IC5.34; no longer IC4.35, IC5.2
- net GND: now also C6.2, C7.2, C8.2, IC1.4, IC4.2, IC5.1, IC5.15, IC5.38, R15.1, T1.2, TP2.TP; no longer C17.2, IC1.58, IC4.1, IC4.15, IC4.38, IC5.13, IC5.22
- net N$5: now also C4.1; no longer C13.1
- net OLED_I2C3_SCL: now also R7.1; no longer R8.1
- net OLED_I2C3_SDA: now also R6.1; no longer R7.1
- net RX1: now also IC5.17; no longer IC4.17
- net SPI2_CS: now also IC1.24; no longer IC1.25
- net TX1: now also IC5.18; no longer IC4.18
Routing:
- net 3.3V: track 237.3 -> 201.2 mm
- net 5V: track 0.00 -> 36.1 mm, vias 0 -> 2
- net POS_DOWN: track 0.00 -> 34.1 mm, vias 0 -> 1
- net POS_5: track 29.4 -> 0.00 mm, vias 1 -> 0
- net POS_1: track 24.9 -> 0.00 mm, vias 1 -> 0
- net 2.8V: track 0.00 -> 23.8 mm, vias 0 -> 2
- net POS_4: track 22.7 -> 0.00 mm, vias 1 -> 0
- net POS_CENTER: track 0.00 -> 21.6 mm, vias 0 -> 1
- net POS_RIGHT: track 0.00 -> 20.1 mm
- net POS_3: track 18.0 -> 0.00 mm, vias 1 -> 0
- net POS_2: track 16.0 -> 0.00 mm, vias 1 -> 0
- net ESP_UART3_TX: track 26.6 -> 12.2 mm
- net FAN: track 0.00 -> 14.3 mm, vias 0 -> 2
- net POS_UP: track 0.00 -> 14.2 mm
- net ESP_UART3_RX: track 25.5 -> 11.7 mm, vias 3 -> 1
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Other:
- board text added: "1"
- board text added: "5V"
- board text added: "A1"
- board text added: "A2"
- board text added: "Buz"
- board text added: "DTR"
- board text added: "Gnd"
- board text added: "JRp"
- board text added: "JRpin5"
- board text added: "RTS"
- board text added: "SRx"
- board text added: "STx"
- board text added: "U1-RX"
- board text added: "U1-TX"
- board text added: "v0.42 rev00"
- board text removed: "v0.31 rev00"
