File: olliw-stm32-based/tx-module-02/mLRS-tx-dualE28-top-v042.sch (EAGLE design)
At the start: 42 parts, among them IC1 STM32G491RC-TQPF64, IC2 E28-2G4M27S, IC3 E28-2G4M27S, IC4 ESP-TTG0-MICROESP32-TTGO-MICRO, IC5 BT HC06, Q1 CSTCE8M00G55-R0, SW1 JOYSTICK-5WAY

Commit message: tx-module02, E28dual board updated to v042 design
Parts:
- removed C17: 10u, rcl:C-EUC0603
- removed PH-BOTCON1, PH-BOTCON2: PINHEAD_3X1WITHBORDER, # stdlib:PINHEAD_3X1WITHBORDER
- removed R8: 2.2k, rcl:R-EU_R0402
- added C6, C8: 100n, rcl:C-EUC0402
- added C7: 10u, rcl:C-EUC0603
- added D2: BAT54J, diode:DIODE-SOD110-R
- added PH-CON1, PH-CON2: PINHEAD_3X1WITHBORDER, # stdlib:PINHEAD_3X1WITHBORDER
- added PH-CON2B: PINHEAD_2X1, # stdlib:PINHEAD_2X1
- added R10, R13: 4.7k, rcl:R-EU_R0402
- added R11, R6: 2.2k, rcl:R-EU_R0402
- added R12: 1k, rcl:R-EU_R0402
- added R14, R15: 10k, rcl:R-EU_R0402
- added T1: FET-NSOT23, # stdlib:FET-NSOT23
- added TP1, TP2, TP3: TPB1,27, testpad:TPB1,27
- C1: device rcl:C-EUC0603 -> rcl:C-EUC0402
- C13: value 100n -> 10u; device rcl:C-EUC0402 -> rcl:C-EUC0603
- C15: value 10u -> 100n; device rcl:C-EUC0603 -> rcl:C-EUC0402
- C16: device rcl:C-EUC0402 -> rcl:C-EUC0603
- C2: value 100n -> 47u; device rcl:C-EUC0603 -> rcl:C-EUC1210
- C3: value 100n -> 47u; device rcl:C-EUC0402 -> rcl:C-EUC1206K
- C4: value 47u -> 100n; device rcl:C-EUC1210 -> rcl:C-EUC0402
- C5: value 47u -> 10u; device rcl:C-EUC1206K -> rcl:C-EUC0603
- IC4: value ESP-TTG0-MICROESP32-TTGO-MICRO -> VREG-5PIN-EN1SOT-89-5; device # stdlib:ESP-TTG0-MICROESP32-TTGO-MICRO -> # stdlib:VREG-5PIN-EN1SOT-89-5
- IC5: value BT HC06 -> ESP-TTG0-MICROESP32-TTGO-MICRO; device # SerialPortBluetooth:HC06-BASIC -> # stdlib:ESP-TTG0-MICROESP32-TTGO-MICRO
Connections:
- removed net POS_1: IC1PORT_C_H.PC14, SW1.B
- removed net POS_2: IC1PORT_C_H.PC13, SW1.A
- removed net POS_3: IC1PORT_C_H.PC15, SW1.CENTER
- removed net POS_4: IC1PORT_C_L.PC3, SW1.C
- removed net POS_5: IC1PORT_C_L.PC2, SW1.D
- new net 2.8V: C15.1, C16.1, IC4.OUT, IC5.3.3V
- new net 5V: C13.1, C14.1, IC4.EN, IC4.IN, IC4.NC, PH-CON1.1
- new net BUZ-: D2.A, T1.D, TP3.TP
- new net DTR: IC1PORT_C_H.PC14, PH-CON2B.2
- new net FAN: IC1PORT_B_L.PB5, R14.1, TP1.TP
- new net N$2: R14.2, R15.2, T1.G
- new net POS_CENTER: IC1PORT_C_H.PC13, SW1.CENTER
- new net POS_DOWN: IC1PORT_C_L.PC2, R12.2, R13.1, SW1.D
- new net POS_LEFT: R11.2, R12.1, SW1.C
- new net POS_RIGHT: R10.2, R11.1, SW1.B
- new net POS_UP: R10.1, SW1.A
- new net RTS: IC1PORT_C_L.PC3, PH-CON2B.1
- net 3.3V: now also C6.1, C7.1, C8.1, D2.C, IC1AN_POWER.VREF+, R13.2, R6.2; no longer C14.1, C15.1, C16.1, C17.1, C4.1, IC4.3.3V, IC5.3V3, R8.2
- net BUZZER: now also PH-CON1.3; no longer PH-BOTCON1.3
- net ESP_GPIO0: now also IC1PORT_B_L.PB1, IC5.IO0; no longer IC1PORT_B_L.PB0, IC4.IO0
- net ESP_LED: now also IC5.IO13; no longer IC4.IO13
- net ESP_RESET: now also IC5.RST/EN; no longer IC4.RST/EN
- net ESP_UART3_RX: now also IC5.TXD0; no longer IC4.RXD0, IC5.TX
- net ESP_UART3_TX: now also IC5.RXD0; no longer IC4.TXD0, IC5.RX
- net GND: now also C6.2, C7.2, C8.2, IC1PORT_C_H.PC15, IC5.GND@1, IC5.GND@2, PH-CON1.5, PH-CON2.5, R15.1, T1.S, TP2.TP; no longer C17.2, IC1PORT_B_L.PB5, IC4.GND@1, IC4.GND@2, IC5.GND2, PH-BOTCON1.5, PH-BOTCON2.5
- net N$5: now also C4.1; no longer C13.1
- net OLED_I2C3_SCL: now also R7.1; no longer R8.1
- net OLED_I2C3_SDA: now also R6.1; no longer R7.1
- net RX1: now also IC5.I09/SD2/U1RX; no longer IC4.I09/SD2/U1RX
- net SPI2_CS: now also IC1PORT_B_L.PB0; no longer IC1PORT_B_L.PB1
- net TX1: now also IC5.IO10/SD3/U1TX; no longer IC4.IO10/SD3/U1TX
- net USB_UART1_RX: now also PH-CON2.3; no longer PH-BOTCON2.3
- net USB_UART1_TX: now also PH-CON2.1; no longer PH-BOTCON2.1
Other:
- note added: "0 V"
- note added: "0.6 V"
- note added: "1.3 V"
- note added: "2.1 V"
- note added: "26. Apr. 2023"
- note added: "Schaltplan v0.42"
- note added: "dummy"
- note removed: "9. Mai. 2022"
- note removed: "Schaltplan v0.31"
- moved on the sheet: C1, C13, C14, C15, C16, C2, C3, C4, C5, IC2, IC3, R7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
