File: olliw-stm32-based/rx-tx-E77-E22-dual-easysolder/mLRS-rx-tx-E77-E22-dual-easysolder-v011.brd (EAGLE design)
At the start: 46.4 x 23.5 mm, 18 parts, among them IC1 LD1117AV33, IC2 E77-900M22S, IC3 E28-SX, SW1 BUTTON6X3.5

Commit message: E77 easy solder , dual/diversity and dual band, v0.11
Parts:
- IC3: value E28-SX -> E22-900M22S; device # stdlib:E28-2G4M27SX -> # stdlib:E22-900M22S
- PH1: value PINHEAD_4X1WITHOUT -> PINHEAD_5X1WITHOUT; device # stdlib:PINHEAD_4X1_WO -> # stdlib:PINHEAD_5X1_WO
- moved IC3 4.76 mm to (11.4, 11.9)
- moved PH1 1.12 mm to (12.7, 22.2)
- moved C6 0.79 mm to (16.7, 21.7)
- moved C5 0.63 mm to (22.9, 21.7)
Connections:
- new net SWRST: IC2.17, PH1.1
- net 3.3V: now also IC3.9, PH1.2; no longer IC3.1, PH1.1
- net BUTTON: now also IC2.8; no longer IC2.25
- net GND: now also IC3.1, IC3.11, IC3.12, IC3.20, IC3.22, IC3.3, IC3.4, IC3.5, PH1.4; no longer IC3.16, IC3.7, PH1.3
- net SPI1_CS: now also IC2.22, IC3.19; no longer IC2.23, IC3.6
- net SPI1_MISO: now also IC3.16; no longer IC3.3
- net SPI1_MOSI: now also IC3.17; no longer IC3.4
- net SPI1_SCK: now also IC3.18; no longer IC3.5
- net SWCLK: now also PH1.3; no longer PH1.2
- net SWDIO: now also PH1.5; no longer PH1.4
- net SX2_BUSY: now also IC2.25, IC3.14; no longer IC2.7, IC3.12
- net SX2_DIO: now also IC2.26; no longer IC2.6
- net SX2_RESET: now also IC2.23, IC3.15; no longer IC2.8, IC3.11
- net SX2_RX_EN: now also IC2.7, IC3.6; no longer IC2.22, IC3.8
- net SX2_TX_EN: now also IC2.6, IC3.7; no longer IC2.11, IC3.9
Routing:
- net SWRST: track 0.00 -> 24.1 mm, vias 0 -> 1
- net BUTTON: track 36.9 -> 32.6 mm, vias 2 -> 0
- net SX2_RESET: track 4.30 -> 7.59 mm
- net SX2_BUSY: track 4.14 -> 6.37 mm
- net 3.3V: track 57.1 -> 59.0 mm, vias 0 -> 1
- net SPI1_MISO: track 11.6 -> 9.68 mm
- net SWDIO: track 29.7 -> 31.2 mm
- net SPI1_MOSI: track 11.8 -> 10.4 mm
- net SPI1_SCK: track 17.6 -> 16.3 mm
- net SX2_TX_EN: track 4.63 -> 3.40 mm
- net SWCLK: track 29.9 -> 28.7 mm
- net SX2_DIO: track 4.14 -> 5.25 mm
- net SPI1_CS: track 3.82 -> 3.08 mm
Other:
- board text added: "E22"
- board text added: "v0.11 rev00"
- board text removed: "E28"
- board text removed: "dual-band"
- board text removed: "v0.10 rev00"
