File: olliw-stm32-based/rx-tx-E77-E22-dual-easysolder/mLRS-rx-tx-E77-E22-dual-easysolder-v011.sch (EAGLE design)
At the start: 18 parts, among them IC1 LD1117AV33, IC2 E77-900M22S, IC3 E28-SX, SW1 BUTTON6X3.5

Commit message: E77 easy solder , dual/diversity and dual band, v0.11
Parts:
- IC3: value E28-SX -> E22-900M22S; device # stdlib:E28-SX -> # stdlib:E22-900M22S
- PH1: value PINHEAD_4X1WITHOUT -> PINHEAD_5X1WITHOUT; device # stdlib:PINHEAD_4X1WITHOUT -> # stdlib:PINHEAD_5X1WITHOUT
Connections:
- new net SWRST: IC2.NRESET, PH1.1
- net 3.3V: now also PH1.2; no longer PH1.1
- net BUTTON: now also IC2.PA1; no longer IC2.PA15
- net GND: now also PH1.4; no longer PH1.3
- net SPI1_CS: now also IC2.PB12, IC3.CS; no longer IC2.PB2, IC3.CS/CTS
- net SPI1_MISO: now also IC3.MISO; no longer IC3.MISO/TX
- net SPI1_MOSI: now also IC3.MOSI; no longer IC3.MOSI/RX
- net SPI1_SCK: now also IC3.SCK; no longer IC3.SCK/RTS
- net SWCLK: now also PH1.3; no longer PH1.2
- net SWDIO: now also PH1.5; no longer PH1.4
- net SX2_BUSY: now also IC2.PA15; no longer IC2.PA0
- net SX2_DIO: now also IC2.PC13; no longer IC2.PB8
- net SX2_RESET: now also IC2.PB2; no longer IC2.PA1
- net SX2_RX_EN: now also IC2.PA0; no longer IC2.PB12
- net SX2_TX_EN: now also IC2.PB8; no longer IC2.PA4
Other:
- note added: "9. Mai 2024"
- note added: "Notes: - C5, C6, E22 are needed only for diversity - If used as tx module, then in the software Tx/Rx must be swapped. That way S becomes the IN (input) signal."
- note added: "Schaltplan v0.11"
- note added: "mLRS E77 E22 easysolder"
- note removed: "1. Mai 2023"
- note removed: "Notes: - In the software Tx/Rx must be swapped. That way S is also the signal (input) when used as tx module."
- note removed: "Schaltplan v0.10"
- note removed: "mLRS E77 E28 easysolder"
- moved on the sheet: IC3
