File: olliw-stm32-based/rx-tx-E77-E28-dualband-easysolder/mLRS-rx-tx-E77-E28-dualband-easysolder-v011.brd (EAGLE design)
At the start: 46.4 x 23.5 mm, 18 parts, among them IC1 LD1117AV33, IC2 E77-900M22S, IC3 E22-900M22S, SW1 BUTTON6X3.5

Commit message: E77 easy solder , dual/diversity and dual band, v0.11
Parts:
- IC3: value E22-900M22S -> E28-SX; device # stdlib:E22-900M22S -> # stdlib:E28-2G4M27SX
- PH1: value PINHEAD_4X1WITHOUT -> PINHEAD_5X1WITHOUT; device # stdlib:PINHEAD_4X1_WO -> # stdlib:PINHEAD_5X1_WO
- moved IC3 4.77 mm to (16.2, 11.7)
- moved PH1 1.12 mm to (12.7, 22.2)
- moved C6 0.79 mm to (16.7, 21.7)
- moved C5 0.63 mm to (22.9, 21.7)
Connections:
- new net SWRST: IC2.17, PH1.1
- net 3.3V: now also IC3.1, PH1.2; no longer IC3.9, PH1.1
- net BUTTON: now also IC2.25; no longer IC2.8
- net GND: now also IC3.16, IC3.7, PH1.4; no longer IC3.1, IC3.11, IC3.12, IC3.20, IC3.22, IC3.3, IC3.4, IC3.5, PH1.3
- net SPI1_CS: now also IC2.23, IC3.6; no longer IC2.22, IC3.19
- net SPI1_MISO: now also IC3.3; no longer IC3.16
- net SPI1_MOSI: now also IC3.4; no longer IC3.17
- net SPI1_SCK: now also IC3.5; no longer IC3.18
- net SWCLK: now also PH1.3; no longer PH1.2
- net SWDIO: now also PH1.5; no longer PH1.4
- net SX2_BUSY: now also IC2.7, IC3.12; no longer IC2.25, IC3.14
- net SX2_DIO: now also IC2.6; no longer IC2.26
- net SX2_RESET: now also IC2.8, IC3.11; no longer IC2.23, IC3.15
- net SX2_RX_EN: now also IC2.22, IC3.8; no longer IC2.7, IC3.6
- net SX2_TX_EN: now also IC2.11, IC3.9; no longer IC2.6, IC3.7
Routing:
- net SWRST: track 0.00 -> 24.5 mm, vias 0 -> 1
- net BUTTON: track 32.6 -> 36.9 mm, vias 0 -> 2
- net SX2_RESET: track 7.59 -> 4.14 mm
- net 3.3V: track 56.0 -> 59.2 mm, vias 0 -> 1
- net SX2_BUSY: track 6.37 -> 3.98 mm
- net SPI1_MISO: track 9.68 -> 11.8 mm
- net SPI1_MOSI: track 10.4 -> 12.0 mm
- net SPI1_SCK: track 16.3 -> 17.7 mm
- net SX2_DIO: track 5.25 -> 3.98 mm
- net SWDIO: track 29.7 -> 30.9 mm
- net SX2_TX_EN: track 3.40 -> 4.50 mm
- net SPI1_CS: track 3.08 -> 3.98 mm
Other:
- board text added: "E28"
- board text added: "dual-band"
- board text added: "v0.11"
- board text removed: "E22"
- board text removed: "v0.10 rev00"
